Commit message: added the docker

File: src/av_gazebo_bringup/urdf/ego_vehicle.urdf.xacro (robot description, xacro)
@@ -13,5 +13,5 @@
       <origin xyz="0 0 0" rpy="0 0 0"/>
       <geometry>
-        <mesh filename="file:///home/nk/.gazebo/models/suv/meshes/suv.obj" scale="0.15 0.15 0.15"/>
+        <mesh filename="file:///root/.gazebo/models/suv/meshes/suv.obj" scale="0.15 0.15 0.15"/>
       </geometry>
     </visual>
